File: ESQUEMA_OG.kicad_sch (KiCad schematic)
At the start: 17 parts, among them U1 ESP32-DEVKIT-V1, U2 ESP32-CAM

Commit message: PCB primera versión de prueba
Parts:
- removed J_CONSOLA_ESP1, J_Interruptor1, J_RELE_PUERTA1, J_RELE_TIMBRE1: 0, Resistor_THT:R_Axial_DIN0207_L6.3mm_D2.5mm_P5.08mm_Vertical, symbol Device:R
- removed J_IRQ_1, J_IRQ_2: Conn_01x01_Socket, Connector_PinSocket_2.54mm:PinSocket_1x01_P2.54mm_Vertical, symbol Connector:Conn_01x01_Socket
Connections:
- net at RELE_PUERTA1.1 (Pin_1): now also U1.22 (D33)
- net at U1.11 (D21): now also PN532.7 (IRQ)
- net at INTERRUPTOR_TIMBRE1.2 (Pin_2): now also U1.23 (D25)
- net at U1.13 (TX0): now also CONSOLA_ESP32.1 (Pin_1)
- net at U1.21 (D32): now also RELE_TIMBRE1.1 (Pin_1)
Other:
- moved on the sheet: CONSOLA_ESP32
