File: PCB/PCB.kicad_pcb (KiCad board)
At the start: 2 copper layers, 17 parts, among them U1 ESP32-DEVKIT-V1, U2 ESP32-CAM

Commit message: Version de prueba para gittear de la RPI
Parts:
- added J_RST_1: Conn_01x01_Socket, Connector_PinSocket_2.54mm:PinSocket_1x01_P2.54mm_Vertical, F.Cu at (168.0, 108.5)
- added J_RST_2: Conn_01x01_Socket, Connector_PinSocket_2.54mm:PinSocket_1x01_P2.54mm_Vertical, F.Cu at (155.5, 70.0)
- PN532: value Conn_01x07 -> PN532-Adafruit; footprint Connector_PinSocket_2.54mm:PinSocket_1x07_P2.54mm_Vertical -> Connector_PinHeader_2.54mm:PinHeader_1x08_P2.54mm_Vertical
- moved J_IRQ_1 21.1 mm to (163.5, 108.5)
- moved CONSOLA_ESP32 16.0 mm to (168.5, 83.2)
- moved J_IRQ_2 15.9 mm to (155.5, 80.5)
- moved USB1 14.8 mm to (111.9, 121.0)
- moved PN532 14.2 mm to (154.5, 118.5)
- moved J_CONSOLA_ESP1 12.6 mm to (157.0, 75.0), turned to 0 degrees
- moved CONSOLA_ESPCAM1 7.52 mm to (177.5, 41.7)
- moved J_Interruptor1 6.57 mm to (116.4, 90.1)
- moved INTERRUPTOR_TIMBRE1 6.12 mm to (95.3, 117.5)
- moved J_RELE_TIMBRE1 5.94 mm to (111.7, 65.5)
- moved J_RELE_PUERTA1 5.77 mm to (112.2, 81.0)
- moved U1 5.59 mm to (137.5, 88.5)
- moved C1 5.02 mm to (171.0, 71.0), turned to 0 degrees
- moved U2 3.12 mm to (158.9, 46.5)
- moved RELE_TIMBRE1 2.86 mm to (93.1, 65.7)
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Connections:
- PN532 pad 5: +5V -> Net-(J_IRQ_1-Pin_1)
- PN532 pad 6: GND -> Net-(J_RST_1-Pin_1)
- PN532 pad 7: Net-(J_IRQ_1-Pin_1) -> GND
- U1 pad 14: unconnected-(U1-D22-Pad14) -> Net-(J_RST_2-Pin_1)
Routing:
- net +5V: track 315.5 -> 247.6 mm
- net Net-(RELE_TIMBRE1-Pin_1): track 20.9 -> 0.00 mm
- net Net-(PN532-SS): track 62.3 -> 49.8 mm
- net Net-(J_IRQ_2-Pin_1): track 17.3 -> 6.08 mm
- net Net-(J_RST_1-Pin_1): track 0.00 -> 10.3 mm
- net Net-(CONSOLA_ESP32-Pin_1): track 19.6 -> 10.9 mm
- net Net-(PN532-SCK): track 44.3 -> 37.4 mm
- net Net-(PN532-MISO): track 47.8 -> 41.0 mm
- net Net-(MOD1-DI): track 73.8 -> 67.1 mm
- net Net-(U1-TX0): track 13.3 -> 7.41 mm
- net Net-(J_RST_2-Pin_1): track 0.00 -> 5.71 mm
- net Net-(CONSOLA_ESPCAM1-Pin_1): track 38.1 -> 33.7 mm
- net Net-(MOD1-RO): track 59.4 -> 55.3 mm
- net Net-(MOD1-DE): track 57.8 -> 53.8 mm
- net Net-(U1-D25): track 8.59 -> 4.91 mm
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- added copper zone on B.Cu, net GND
- removed copper zone on F.Cu, net GND
Other:
- board outline added: 90 x 90 mm
