File: PCB/PCB.kicad_sch (KiCad schematic)
At the start: 17 parts, among them U1 ESP32-DEVKIT-V1, U2 ESP32-CAM

Commit message: Version de prueba para gittear de la RPI
Parts:
- added J_RST_1, J_RST_2: Conn_01x01_Socket, Connector_PinSocket_2.54mm:PinSocket_1x01_P2.54mm_Vertical, symbol Connector:Conn_01x01_Socket
- PN532: value Conn_01x07 -> PN532-Adafruit; footprint Connector_PinSocket_2.54mm:PinSocket_1x07_P2.54mm_Vertical -> Connector_PinHeader_2.54mm:PinHeader_1x08_P2.54mm_Vertical
Connections:
- net +5V: now also PN532.8 (5V); no longer PN532.5 (VCC)
- net GND: now also PN532.7 (GND); no longer PN532.6 (GND)
- net at J_IRQ_1.1 (Pin_1): now also PN532.5 (IRQ); no longer PN532.7 (IRQ)
- net at U1.14 (D22): now also J_RST_2.1 (Pin_1)
- new net: J_RST_1.1 (Pin_1), PN532.6 (RST)
Other:
- moved on the sheet: J_IRQ_1
